Commit message: Environnement without physics

File: Assets/URDF/Panda_Robot/robots/hand.urdf (robot description, URDF)
Before this commit: robot hand, 3 links, 2 joints
Links:
- link panda_hand: geometry collision mesh filename=meshes/collision/hand.stl; visual mesh filename=meshes/visual/hand.dae
- link panda_leftfinger: geometry collision mesh filename=meshes/collision/finger.stl; visual mesh filename=meshes/visual/finger.dae
- link panda_rightfinger: geometry collision mesh filename=meshes/collision/finger.stl; visual mesh filename=meshes/visual/finger.dae
